Commit message: Extend UR15 URDF with fixed two-finger gripper and tool camera links; add gripper STL location doc

File: Chalmers/Kandidatarbete/UR15_ROS2_Integration/Assets/robot/ur15 (copy).urdf (robot description, URDF)
Before this commit: robot ur15_unity_clean, 9 links, 8 joints
Links:
- added link gripper_base_link; collision mesh filename=package://ur_description/meshes/gripper/gripper_base.stl; visual mesh filename=package://ur_description/meshes/gripper/gripper_base.stl
- added link left_finger_link; collision mesh filename=package://ur_description/meshes/gripper/left_finger.stl; visual mesh filename=package://ur_description/meshes/gripper/left_finger.stl
- added link right_finger_link; collision mesh filename=package://ur_description/meshes/gripper/right_finger.stl; visual mesh filename=package://ur_description/meshes/gripper/right_finger.stl
- added link tool0; collision cylinder length=0.08 radius=0.02; visual cylinder length=0.08 radius=0.02
- added link tool_camera_link; collision box size=0.035 0.025 0.02; visual box size=0.035 0.025 0.02
Joints:
- added joint gripper_base_fixed: type fixed, parent tool0, child gripper_base_link, origin xyz=0 0 0.06 rpy=0 0 0
- added joint left_finger_fixed: type fixed, parent gripper_base_link, child left_finger_link, origin xyz=0 0.03 0.04 rpy=0 0 0
- added joint right_finger_fixed: type fixed, parent gripper_base_link, child right_finger_link, origin xyz=0 -0.03 0.04 rpy=0 0 0
- added joint tool0_fixed: type fixed, parent wrist_3_link, child tool0, origin xyz=0 0 0.12 rpy=0 0 0
- added joint tool_camera_fixed: type fixed, parent gripper_base_link, child tool_camera_link, origin xyz=0 0 0 rpy=0 0 0

Commit message: Wire gripper URDF to pushed STL names and make finger joints revolute

File: Chalmers/Kandidatarbete/UR15_ROS2_Integration/Assets/robot/ur15 (copy).urdf (robot description, URDF)
Before this commit: robot ur15_unity_clean, 14 links, 13 joints
Links:
- link gripper_base_link: geometry collision mesh filename=package://ur_description/meshes/gripper/gripper_base_with_p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; visual mesh filename=package://ur_description/meshes/gripper/gripper_base_with_p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
- link left_finger_link: geometry collision mesh filename=package://ur_description/meshes/gripper/finger.stl; visual mesh filename=package://ur_description/meshes/gripper/finger.stl
- link right_finger_link: geometry collision mesh filename=package://ur_description/meshes/gripper/finger.stl; visual mesh filename=package://ur_description/meshes/gripper/finger.stl
Joints:
- removed joint left_finger_fixed
- removed joint right_finger_fixed
- added joint left_finger_joint: type revolute, parent gripper_base_link, child left_finger_link, origin xyz=0 0.03 0.04 rpy=0 0 0, axis 0 0 1, limit lower=0.0 upper=0.7 effort=20 velocity=1.0
- added joint right_finger_joint: type revolute, parent gripper_base_link, child right_finger_link, origin xyz=0 -0.03 0.04 rpy=0 0 0, axis 0 0 1, limit lower=-0.7 upper=0.0 effort=20 velocity=1.0

Commit message: Scale gripper meshes from mm to meters in URDF (0.001)

File: Chalmers/Kandidatarbete/UR15_ROS2_Integration/Assets/robot/ur15 (copy).urdf (robot description, URDF)
Before this commit: robot ur15_unity_clean, 14 links, 13 joints
Links:
- link gripper_base_link: geometry collision mesh filename=package://ur_description/meshes/gripper/gripper_base_with_p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 scale=0.001 0.001 0.001; visual mesh filename=package://ur_description/meshes/gripper/gripper_base_with_p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 scale=0.001 0.001 0.001
- link left_finger_link: geometry collision mesh filename=package://ur_description/meshes/gripper/finger.stl scale=0.001 0.001 0.001; visual mesh filename=package://ur_description/meshes/gripper/finger.stl scale=0.001 0.001 0.001
- link right_finger_link: geometry collision mesh filename=package://ur_description/meshes/gripper/finger.stl scale=0.001 0.001 0.001; visual mesh filename=package://ur_description/meshes/gripper/finger.stl scale=0.001 0.001 0.001

Commit message: Tune gripper alignment: rotate base + adjust mount/finger offsets

File: Chalmers/Kandidatarbete/UR15_ROS2_Integration/Assets/robot/ur15 (copy).urdf (robot description, URDF)
Before this commit: robot ur15_unity_clean, 14 links, 13 joints
Joints:
- joint gripper_base_fixed: origin xyz=0 0 0.06 rpy=0 0 0 -> xyz=0 0 0.085 rpy=0 1.57079632679 0
- joint left_finger_joint: origin xyz=0 0.03 0.04 rpy=0 0 0 -> xyz=0.01 0.032 0.03 rpy=0 0 0
- joint right_finger_joint: origin xyz=0 -0.03 0.04 rpy=0 0 0 -> xyz=0.01 -0.032 0.03 rpy=0 0 0

Commit message: Create direct wrist-mounted gripper variant: remove tool0 and rotate gripper/fingers +90deg around Z

File: Chalmers/Kandidatarbete/UR15_ROS2_Integration/Assets/robot/ur15 (copy).urdf (robot description, URDF)
Before this commit: robot ur15_unity_clean, 14 links, 13 joints
Links:
- removed link tool0
Joints:
- removed joint tool0_fixed
- joint gripper_base_fixed: origin xyz=0 0 0.085 rpy=0 1.57079632679 0 -> xyz=0 0 0.205 rpy=0 1.57079632679 1.57079632679; parent tool0 -> wrist_3_link
- joint left_finger_joint: origin xyz=0.01 0.032 0.03 rpy=0 0 0 -> xyz=0.01 0.032 0.03 rpy=0 0 1.57079632679
- joint right_finger_joint: origin xyz=0.01 -0.032 0.03 rpy=0 0 0 -> xyz=0.01 -0.032 0.03 rpy=0 0 1.57079632679

Commit message: WIP: gripper base aligned, finger alignment pending

File: Chalmers/Kandidatarbete/UR15_ROS2_Integration/Assets/robot/ur15 (copy).urdf (robot description, URDF)
Before this commit: robot ur15_unity_clean, 13 links, 12 joints
Joints:
- joint gripper_base_fixed: origin xyz=0 0 0.205 rpy=0 1.57079632679 1.57079632679 -> xyz=0 0 0 rpy=0 -1.57079632679 0
- joint left_finger_joint: origin xyz=0.01 0.032 0.03 rpy=0 0 1.57079632679 -> xyz=0 0.03 0.00 rpy=0 0 0
- joint right_finger_joint: axis 0 0 1 -> 0 0 -1; origin xyz=0.01 -0.032 0.03 rpy=0 0 1.57079632679 -> xyz=0 -0.03 0.00 rpy=0 0 0

Commit message: Normalize finger frames: mirror via right joint rpy, unify axes/limits, and tune finger offsets

File: Chalmers/Kandidatarbete/UR15_ROS2_Integration/Assets/robot/ur15 (copy).urdf (robot description, URDF)
Before this commit: robot ur15_unity_clean, 13 links, 12 joints
Joints:
- joint left_finger_joint: origin xyz=0 0.03 0.00 rpy=0 0 0 -> xyz=0.012 0.03 0.00 rpy=0 0 0
- joint right_finger_joint: axis 0 0 -1 -> 0 0 1; limit lower=-0.7 upper=0.0 effort=20 velocity=1.0 -> lower=0.0 upper=0.7 effort=20 velocity=1.0; origin xyz=0 -0.03 0.00 rpy=0 0 0 -> xyz=0.012 -0.03 0.00 rpy=0 0 3.14159265359

Commit message: Finalize UR15 + gripper alignment baseline (manual calibrated)

File: Chalmers/Kandidatarbete/UR15_ROS2_Integration/Assets/robot/ur15 (copy).urdf (robot description, URDF)
Before this commit: robot ur15_unity_clean, 13 links, 12 joints
Joints:
- joint right_finger_joint: origin xyz=0.012 -0.03 0.00 rpy=0 0 3.14159265359 -> xyz=0.012 -0.03 0.00 rpy=0 0 0

Commit message: Improve gripper finger motion direction and reposition tool camera mount

File: Chalmers/Kandidatarbete/UR15_ROS2_Integration/Assets/robot/ur15 (copy).urdf (robot description, URDF)
Before this commit: robot ur15_unity_clean, 13 links, 12 joints
Joints:
- joint right_finger_joint: axis 0 0 1 -> 0 0 -1
- joint tool_camera_fixed: origin xyz=0 0 0 rpy=0 0 0 -> xyz=0.11 0 0.055 rpy=0 -1.57079632679 0

Commit message: Remove tool camera link/joint from UR15 URDF for now

File: Chalmers/Kandidatarbete/UR15_ROS2_Integration/Assets/robot/ur15 (copy).urdf (robot description, URDF)
Before this commit: robot ur15_unity_clean, 13 links, 12 joints
Links:
- removed link tool_camera_link
Joints:
- removed joint tool_camera_fixed

Commit message: Apply default joint params in URDF: limits +/-180deg, damping 200, safety/stiffness 800

File: Chalmers/Kandidatarbete/UR15_ROS2_Integration/Assets/robot/ur15 (copy).urdf (robot description, URDF)
Before this commit: robot ur15_unity_clean, 12 links, 11 joints
Joints:
- joint elbow_joint: limit (none) -> lower=-3.14159265359 upper=3.14159265359 effort=800 velocity=200
- joint left_finger_joint: limit lower=0.0 upper=0.7 effort=20 velocity=1.0 -> lower=-3.14159265359 upper=3.14159265359 effort=800 velocity=200
- joint right_finger_joint: limit lower=0.0 upper=0.7 effort=20 velocity=1.0 -> lower=-3.14159265359 upper=3.14159265359 effort=800 velocity=200
- joint shoulder_lift_joint: limit (none) -> lower=-3.14159265359 upper=3.14159265359 effort=800 velocity=200
- joint shoulder_pan_joint: limit (none) -> lower=-3.14159265359 upper=3.14159265359 effort=800 velocity=200
- joint wrist_1_joint: limit (none) -> lower=-3.14159265359 upper=3.14159265359 effort=800 velocity=200
- joint wrist_2_joint: limit (none) -> lower=-3.14159265359 upper=3.14159265359 effort=800 velocity=200
- joint wrist_3_joint: limit (none) -> lower=-3.14159265359 upper=3.14159265359 effort=800 velocity=200

Commit message: Set realistic finger joint limits/drives in URDF (0..0.7, effort 300, damping 20)

File: Chalmers/Kandidatarbete/UR15_ROS2_Integration/Assets/robot/ur15 (copy).urdf (robot description, URDF)
Before this commit: robot ur15_unity_clean, 12 links, 11 joints
Joints:
- joint left_finger_joint: limit lower=-3.14159265359 upper=3.14159265359 effort=800 velocity=200 -> lower=0.0 upper=0.7 effort=300 velocity=2.0
- joint right_finger_joint: limit lower=-3.14159265359 upper=3.14159265359 effort=800 velocity=200 -> lower=0.0 upper=0.7 effort=300 velocity=2.0

Commit message: Fix finger motion to linear: prismatic joints + trajectory driver support for meter targets

File: Chalmers/Kandidatarbete/UR15_ROS2_Integration/Assets/robot/ur15 (copy).urdf (robot description, URDF)
Before this commit: robot ur15_unity_clean, 12 links, 11 joints
Joints:
- joint left_finger_joint: axis 0 0 1 -> 0 1 0; limit lower=0.0 upper=0.7 effort=300 velocity=2.0 -> lower=0.0 upper=0.02 effort=300 velocity=0.05; type revolute -> prismatic
- joint right_finger_joint: axis 0 0 -1 -> 0 -1 0; limit lower=0.0 upper=0.7 effort=300 velocity=2.0 -> lower=0.0 upper=0.02 effort=300 velocity=0.05; type revolute -> prismatic

Commit message: Fix finger frames for linear gripper motion: symmetric mesh origins and X-axis prismatic joints

File: Chalmers/Kandidatarbete/UR15_ROS2_Integration/Assets/robot/ur15 (copy).urdf (robot description, URDF)
Before this commit: robot ur15_unity_clean, 12 links, 11 joints
Joints:
- joint left_finger_joint: axis 0 1 0 -> 1 0 0
- joint right_finger_joint: axis 0 -1 0 -> -1 0 0

Commit message: Revert right finger placement; only adjust prismatic movement direction axes

File: Chalmers/Kandidatarbete/UR15_ROS2_Integration/Assets/robot/ur15 (copy).urdf (robot description, URDF)
Before this commit: robot ur15_unity_clean, 12 links, 11 joints
Joints:
- joint left_finger_joint: axis 1 0 0 -> 0 1 0
- joint right_finger_joint: axis -1 0 0 -> 0 -1 0

Commit message: WIP: stream resolution runtime issue

File: Chalmers/Kandidatarbete/UR15_ROS2_Integration/Assets/robot/ur15 (copy).urdf (robot description, URDF)
Before this commit: robot ur15_unity_clean, 12 links, 11 joints
Joints:
- joint left_finger_joint: axis 0 1 0 -> 0 0 -1; limit lower=0.0 upper=0.02 effort=300 velocity=0.05 -> lower=0.0 upper=20 effort=2000 velocity=0.05
- joint right_finger_joint: axis 0 -1 0 -> 0 0 1; limit lower=0.0 upper=0.02 effort=300 velocity=0.05 -> lower=0.0 upper=20 effort=2000 velocity=0.05
