Commit message: Add gripper to ur10e_official and apply UR-style color materials

File: Chalmers/Kandidatarbete/UR15_ROS2_Integration/Assets/robot/ur10e_official.urdf (robot description, URDF)
Before this commit: robot ur10e_robot, 11 links, 10 joints
Links:
- added link gripper_base_link; collision mesh filename=package://ur_description/meshes/gripper/gripper_base_with_p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 scale=0.001 0.001 0.001; visual mesh filename=package://ur_description/meshes/gripper/gripper_base_with_p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 scale=0.001 0.001 0.001
- added link left_finger_link; collision mesh filename=package://ur_description/meshes/gripper/finger.stl scale=0.001 0.001 0.001; visual mesh filename=package://ur_description/meshes/gripper/finger.stl scale=0.001 0.001 0.001
- added link right_finger_link; collision mesh filename=package://ur_description/meshes/gripper/finger.stl scale=0.001 0.001 0.001; visual mesh filename=package://ur_description/meshes/gripper/finger.stl scale=0.001 0.001 0.001
Joints:
- added joint left_finger_joint: type prismatic, parent gripper_base_link, child left_finger_link, origin xyz=0.012 0.03 0.00 rpy=0 0 0, axis 0 1 0, limit lower=0.0 upper=0.06 effort=300 velocity=0.05
- added joint right_finger_joint: type prismatic, parent gripper_base_link, child right_finger_link, origin xyz=0.012 -0.03 0.00 rpy=0 0 0, axis 0 -1 0, limit lower=0.0 upper=0.06 effort=300 velocity=0.05
- added joint tool0-gripper_base_fixed: type fixed, parent tool0, child gripper_base_link, origin xyz=0 0 0 rpy=0 -1.57079632679 0

Commit message: falls over

File: Chalmers/Kandidatarbete/UR15_ROS2_Integration/Assets/robot/ur10e_official.urdf (robot description, URDF)
Before this commit: robot ur10e_robot, 14 links, 13 joints
Joints:
- joint left_finger_joint: axis 0 1 0 -> 0 0 -1
- joint right_finger_joint: axis 0 -1 0 -> 0 0 1
