Commit message: Add prismatic rail joint for UR10e side-to-side motion

File: Chalmers/Kandidatarbete/ros2_ws/src/ur_description/urdf/ur10e_official.urdf (robot description, URDF)
Before this commit: robot ur10e_robot, 14 links, 13 joints
Links:
- added link rail_base_link; collision box size=2.4 0.08 0.08; visual box size=2.4 0.08 0.08
Joints:
- added joint rail_joint: type prismatic, parent rail_base_link, child base_link, origin xyz=0 0 0.04035 rpy=0 0 0, axis 0 1 0, limit lower=-1.0 upper=1.0 effort=2000.0 velocity=0.4
