Commit message: WIP: Unity rail + trajectory debug before pause

File: Chalmers/Kandidatarbete/ros2_ws/install/ur_description/share/ur_description/urdf/ur10e_official.urdf (robot description, URDF)
Before this commit: robot ur10e_robot, 14 links, 13 joints
Links:
- added link rail_base_link; collision box size=2.4 0.08 0.08; visual box size=2.4 0.08 0.08
- added link world
Joints:
- added joint rail_joint: type prismatic, parent rail_base_link, child base_link, origin xyz=0 0 0.04035 rpy=0 0 0, axis 0 1 0, limit lower=-1.0 upper=1.0 effort=2000.0 velocity=0.4
- added joint world_to_rail_base: type fixed, parent world, child rail_base_link, origin xyz=0 0.02 1.6 rpy=1.5707963267948966 0 3.141592653589793

Commit message: WIP: rail constrained target publisher integrated and tested

File: Chalmers/Kandidatarbete/ros2_ws/install/ur_description/share/ur_description/urdf/ur10e_official.urdf (robot description, URDF)
Before this commit: robot ur10e_robot, 16 links, 15 joints
Links:
- link rail_base_link: geometry collision box size=4.65 0.08 0.08; visual box size=4.65 0.08 0.08
Joints:
- joint rail_joint: axis 0 1 0 -> 1 0 0; limit lower=-1.0 upper=1.0 effort=2000.0 velocity=0.4 -> lower=-2.325 upper=2.325 effort=2000.0 velocity=0.4
- joint shoulder_lift_joint: limit lower=-6.283185307179586 upper=6.283185307179586 effort=330.0 velocity=2.0943951023931953 -> lower=-6.283185307179586 upper=6.283185307179586 effort=900.0 velocity=2.0943951023931953
- joint shoulder_pan_joint: limit lower=-6.283185307179586 upper=6.283185307179586 effort=330.0 velocity=2.0943951023931953 -> lower=-6.283185307179586 upper=6.283185307179586 effort=900.0 velocity=2.0943951023931953
