Commit message: Set UR10e world pose to Unity-aligned mount transform

File: Chalmers/Kandidatarbete/UR10e_ROS2_Baseline/Assets/robot/ur10e_official.urdf (robot description, URDF)
Before this commit: robot ur10e_robot, 15 links, 14 joints
Links:
- added link world
Joints:
- added joint world_to_rail_base: type fixed, parent world, child rail_base_link, origin xyz=-0.02 1.6 0 rpy=3.141592653589793 0 1.5707963267948966

Commit message: Set robot base height to 1.6m with neutral world alignment

File: Chalmers/Kandidatarbete/UR10e_ROS2_Baseline/Assets/robot/ur10e_official.urdf (robot description, URDF)
Before this commit: robot ur10e_robot, 16 links, 15 joints
Joints:
- joint world_to_rail_base: origin xyz=-0.02 1.6 0 rpy=3.141592653589793 0 1.5707963267948966 -> xyz=0 0 1.6 rpy=0 0 0

Commit message: Reset world mount to origin with zero rotation

File: Chalmers/Kandidatarbete/UR10e_ROS2_Baseline/Assets/robot/ur10e_official.urdf (robot description, URDF)
Before this commit: robot ur10e_robot, 16 links, 15 joints
Joints:
- joint world_to_rail_base: origin xyz=0 0 1.6 rpy=0 0 0 -> xyz=0 0 0 rpy=0 0 0

Commit message: Set world_to_rail_base using Unity axis mapping

File: Chalmers/Kandidatarbete/UR10e_ROS2_Baseline/Assets/robot/ur10e_official.urdf (robot description, URDF)
Before this commit: robot ur10e_robot, 16 links, 15 joints
Joints:
- joint world_to_rail_base: origin xyz=0 0 0 rpy=0 0 0 -> xyz=0 -0.02 1.6 rpy=0 0 0

Commit message: Rotate mount and apply requested default articulation drive settings

File: Chalmers/Kandidatarbete/UR10e_ROS2_Baseline/Assets/robot/ur10e_official.urdf (robot description, URDF)
Before this commit: robot ur10e_robot, 16 links, 15 joints
Joints:
- joint world_to_rail_base: origin xyz=0 -0.02 1.6 rpy=0 0 0 -> xyz=0 -0.02 1.6 rpy=3.141592653589793 0 1.5707963267948966

Commit message: Adjust mount rotation axes to match Unity orientation mapping

File: Chalmers/Kandidatarbete/UR10e_ROS2_Baseline/Assets/robot/ur10e_official.urdf (robot description, URDF)
Before this commit: robot ur10e_robot, 16 links, 15 joints
Joints:
- joint world_to_rail_base: origin xyz=0 -0.02 1.6 rpy=3.141592653589793 0 1.5707963267948966 -> xyz=0 -0.02 1.6 rpy=1.5707963267948966 3.141592653589793 0

Commit message: Set mount rotation to 180 degrees around Z axis

File: Chalmers/Kandidatarbete/UR10e_ROS2_Baseline/Assets/robot/ur10e_official.urdf (robot description, URDF)
Before this commit: robot ur10e_robot, 16 links, 15 joints
Joints:
- joint world_to_rail_base: origin xyz=0 -0.02 1.6 rpy=1.5707963267948966 3.141592653589793 0 -> xyz=0 -0.02 1.6 rpy=0 0 3.141592653589793

Commit message: Increase mount Z rotation by 90 degrees (to 270 deg)

File: Chalmers/Kandidatarbete/UR10e_ROS2_Baseline/Assets/robot/ur10e_official.urdf (robot description, URDF)
Before this commit: robot ur10e_robot, 16 links, 15 joints
Joints:
- joint world_to_rail_base: origin xyz=0 -0.02 1.6 rpy=0 0 3.141592653589793 -> xyz=0 -0.02 1.6 rpy=0 0 4.71238898038469

Commit message: Add another +90deg on mount Z rotation

File: Chalmers/Kandidatarbete/UR10e_ROS2_Baseline/Assets/robot/ur10e_official.urdf (robot description, URDF)
Before this commit: robot ur10e_robot, 16 links, 15 joints
Joints:
- joint world_to_rail_base: origin xyz=0 -0.02 1.6 rpy=0 0 4.71238898038469 -> xyz=0 -0.02 1.6 rpy=0 0 6.283185307179586

Commit message: Apply +90deg about Unity Z using mapped URDF axis

File: Chalmers/Kandidatarbete/UR10e_ROS2_Baseline/Assets/robot/ur10e_official.urdf (robot description, URDF)
Before this commit: robot ur10e_robot, 16 links, 15 joints
Joints:
- joint world_to_rail_base: origin xyz=0 -0.02 1.6 rpy=0 0 6.283185307179586 -> xyz=0 -0.02 1.6 rpy=1.5707963267948966 0 0

Commit message: Fix Unity URDF mount orientation

File: Chalmers/Kandidatarbete/UR10e_ROS2_Baseline/Assets/robot/ur10e_official.urdf (robot description, URDF)
Before this commit: robot ur10e_robot, 16 links, 15 joints
Joints:
- joint world_to_rail_base: origin xyz=0 -0.02 1.6 rpy=1.5707963267948966 0 0 -> xyz=0 0.02 1.6 rpy=1.5707963267948966 0 3.141592653589793

Commit message: Fix rail_joint axis to move laterally instead of vertical drop

File: Chalmers/Kandidatarbete/UR10e_ROS2_Baseline/Assets/robot/ur10e_official.urdf (robot description, URDF)
Before this commit: robot ur10e_robot, 16 links, 15 joints
Joints:
- joint rail_joint: axis 0 1 0 -> 1 0 0

Commit message: Set rail_joint axis to local Y for correct lateral motion

File: Chalmers/Kandidatarbete/UR10e_ROS2_Baseline/Assets/robot/ur10e_official.urdf (robot description, URDF)
Before this commit: robot ur10e_robot, 16 links, 15 joints
Joints:
- joint rail_joint: axis 1 0 0 -> 0 1 0

Commit message: Stabilize rail control and extend rail travel to 4.65m

File: Chalmers/Kandidatarbete/UR10e_ROS2_Baseline/Assets/robot/ur10e_official.urdf (robot description, URDF)
Before this commit: robot ur10e_robot, 16 links, 15 joints
Joints:
- joint rail_joint: limit lower=-1.0 upper=1.0 effort=2000.0 velocity=0.4 -> lower=-2.325 upper=2.325 effort=2000.0 velocity=0.4

Commit message: Expand rail_base_link geometry to 4.65m to match travel range

File: Chalmers/Kandidatarbete/UR10e_ROS2_Baseline/Assets/robot/ur10e_official.urdf (robot description, URDF)
Before this commit: robot ur10e_robot, 16 links, 15 joints
Links:
- link rail_base_link: geometry collision box size=4.65 0.08 0.08; visual box size=4.65 0.08 0.08

Commit message: Boost base joint effort/damping and set safer default OMPL scaling

File: Chalmers/Kandidatarbete/UR10e_ROS2_Baseline/Assets/robot/ur10e_official.urdf (robot description, URDF)
Before this commit: robot ur10e_robot, 16 links, 15 joints
Joints:
- joint shoulder_pan_joint: limit lower=-6.283185307179586 upper=6.283185307179586 effort=330.0 velocity=2.0943951023931953 -> lower=-6.283185307179586 upper=6.283185307179586 effort=900.0 velocity=2.0943951023931953

Commit message: Strengthen base/shoulder drives and speed up base joint response

File: Chalmers/Kandidatarbete/UR10e_ROS2_Baseline/Assets/robot/ur10e_official.urdf (robot description, URDF)
Before this commit: robot ur10e_robot, 16 links, 15 joints
Joints:
- joint shoulder_lift_joint: limit lower=-6.283185307179586 upper=6.283185307179586 effort=330.0 velocity=2.0943951023931953 -> lower=-6.283185307179586 upper=6.283185307179586 effort=900.0 velocity=2.0943951023931953

Commit message: Inflate rail collision box for safer planning clearance

File: Chalmers/Kandidatarbete/UR10e_ROS2_Baseline/Assets/robot/ur10e_official.urdf (robot description, URDF)
Before this commit: robot ur10e_robot, 16 links, 15 joints
Links:
- link rail_base_link: geometry collision box size=4.65 0.16 0.16; visual box size=4.65 0.08 0.08

Commit message: Tune rail collision inflation to medium size (0.14m)

File: Chalmers/Kandidatarbete/UR10e_ROS2_Baseline/Assets/robot/ur10e_official.urdf (robot description, URDF)
Before this commit: robot ur10e_robot, 16 links, 15 joints
Links:
- link rail_base_link: geometry collision box size=4.65 0.14 0.14; visual box size=4.65 0.08 0.08
